File: PCB/KiCAD/Main (Teensy)/Main (Teensy).kicad_sch (KiCad schematic)
At the start: 158 parts, among them J1 Conn_02x03_Odd_Even, J10 Conn_01x04, J2 Conn_01x02, J3 Conn_01x04, J4 Conn_01x04, J5 Conn_01x02, J6 Conn_01x06, J7 Conn_01x04, J8 Conn_01x02, J9 Conn_01x02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

Commit message: Battery XT60 was reversed
Connections:
- net Earth: now also J2.1 (Pin_1); no longer J2.2 (Pin_2)
- net at F1.1: now also J2.2 (Pin_2); no longer J2.1 (Pin_1)
Other:
- moved on the sheet: J2
Changed lines of the file:
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@@
 	(wire
 		(pts
+			(xy 49.53 186.69) (xy 49.53 187.96)
+		)
+		(stroke
+			(width 0)
+			(type default)
+		)
+	)
+	(wire
+		(pts
 			(xy 49.53 330.2) (xy 49.53 327.66)
 		)
@@
 	(wire
 		(pts
-			(xy 49.53 187.96) (xy 49.53 186.69)
+			(xy 49.53 186.69) (xy 46.99 186.69)
 		)
 		(stroke
@@
 	(wire
 		(pts
-			(xy 49.53 186.69) (xy 48.26 186.69)
-		)
-		(stroke
-			(width 0)
-			(type default)
-		)
-	)
-	(wire
-		(pts
 			(xy 26.67 130.81) (xy 27.94 130.81)
 		)
@@
 	(wire
 		(pts
-			(xy 48.26 184.15) (xy 49.53 184.15)
-		)
-		(stroke
-			(width 0)
-			(type default)
-		)
-	)
-	(wire
-		(pts
 			(xy 140.97 250.19) (xy 142.24 250.19)
 		)
@@
 	(wire
 		(pts
+			(xy 46.99 184.15) (xy 49.53 184.15)
+		)
+		(stroke
+			(width 0)
+			(type default)
+		)
+	)
+	(wire
+		(pts
 			(xy 135.89 261.62) (xy 135.89 233.68)
 		)
@@
 	(symbol
 		(lib_id "Connector_Generic:Conn_01x02")
-		(at 43.18 184.15 0)
-		(mirror y)
+		(at 41.91 186.69 180)
 		(unit 1)
 		(exclude_from_sim no)
@@
 		(dnp no)
 		(property "Reference" "J2"
-			(at 43.18 181.356 0)
+			(at 41.91 189.484 0)
 			(effects
 				(font
@@
 		)
 		(property "Value" "Conn_01x02"
-			(at 43.18 190.5 0)
+			(at 41.91 180.34 0)
 			(effects
 				(font
@@
 		)
 		(property "Footprint" "Connector_AMASS:AMASS_XT60-M_1x02_P7.20mm_Vertical"
-			(at 43.18 184.15 0)
+			(at 41.91 186.69 0)
 			(effects
 				(font
@@
 		)
 		(property "Datasheet" "~"
-			(at 43.18 184.15 0)
+			(at 41.91 186.69 0)
 			(effects
 				(font
@@
 		)
 		(property "Description" "Generic connector, single row, 01x02, script generated (kicad-library-utils/schlib/autogen/connector/)"
-			(at 43.18 184.15 0)
+			(at 41.91 186.69 0)
 			(effects
 				(font
