File: PCB/KiCAD/Main PCB/led_indicators.kicad_sch (KiCad schematic)
At the start: 48 parts

Commit message: New motor controllers for the main PCB
Parts:
- removed D10, D12, D14, D16, D18, D20, D22, D24: BALL_DIR_LED, LED_SMD:LED_0805_2012Metric_Pad1.15x1.40mm_HandSolder, symbol Device:LED
- removed D7: RED_LED, LED_SMD:LED_0805_2012Metric_Pad1.15x1.40mm_HandSolder, symbol Device:LED
- removed R22: 330, Resistor_SMD:R_0805_2012Metric_Pad1.20x1.40mm_HandSolder, symbol Device:R
- removed R25, R27, R29, R31, R33, R35, R37, R39: 130, Resistor_SMD:R_0805_2012Metric_Pad1.20x1.40mm_HandSolder, symbol Device:R
- renumbered D13 to D10, D15 to D11, D17 to D12, D19 to D13, D21 to D14, D23 to D15, D8 to D7, D9 to D8, D11 to D9, R16 to R15, R17 to R16, R18 to R17, R19 to R18, R20 to R19, R21 to R20, R23 to R21, R24 to R22, R26 to R23, R28 to R24, R30 to R25, R32 to R26, R34 to R27, R36 to R28, R38 to R29
Connections:
- net STATUS_GREEN_4_0 renamed STATUS_GREEN_TEENSY_1
- net STATUS_GREEN_4_1 renamed STATUS_GREEN_MAIN
- net STATUS_RED_4_1 renamed STATUS_RED_MAIN
Other:
- moved on the sheet: D10, D11, D12, D13, D14, D15, D7, D8, D9, R21, R22, R23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

Commit message: Added a BNO055 and traced PCB (incomplete, no DRC pass)
Parts:
- renumbered R15 to R30, R16 to R31, R17 to R32, R18 to R33, R19 to R34, R20 to R35, R21 to R36, R22 to R37, R23 to R38, R24 to R39, R25 to R40, R26 to R41, R27 to R42, R28 to R43, R29 to R44
Changed lines of the file:
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@@
 		(on_board yes)
 		(dnp no)
-		(property "Reference" "R16"
+		(property "Reference" "R31"
 			(at 107.95 44.45 0)
 			(effects
@@
 			(project "Main PCB"
 				(path "/2fa7e914-8c49-49b7-a5a9-3cb78b2e953f/61c7190e-5a84-4d72-bf05-2bf9053a9edb"
-					(reference "R16")
+					(reference "R31")
 					(unit 1)
 				)
@@
 		(on_board yes)
 		(dnp no)
-		(property "Reference" "R15"
+		(property "Reference" "R30"
 			(at 107.95 36.83 0)
 			(effects
@@
 			(project "Main PCB"
 				(path "/2fa7e914-8c49-49b7-a5a9-3cb78b2e953f/61c7190e-5a84-4d72-bf05-2bf9053a9edb"
-					(reference "R15")
+					(reference "R30")
 					(unit 1)
 				)
@@
 		(dnp no)
 		(fields_autoplaced yes)
-		(property "Reference" "#PWR052"
+		(property "Reference" "#PWR056"
 			(at 129.54 60.96 0)
 			(effects
@@
 			(project "Main PCB"
 				(path "/2fa7e914-8c49-49b7-a5a9-3cb78b2e953f/61c7190e-5a84-4d72-bf05-2bf9053a9edb"
-					(reference "#PWR052")
+					(reference "#PWR056")
 					(unit 1)
 				)
@@
 		(on_board yes)
 		(dnp no)
-		(property "Reference" "R21"
+		(property "Reference" "R36"
 			(at 107.188 91.948 90)
 			(effects
@@
 			(project "Main PCB"
 				(path "/2fa7e914-8c49-49b7-a5a9-3cb78b2e953f/61c7190e-5a84-4d72-bf05-2bf9053a9edb"
-					(reference "R21")
+					(reference "R36")
 					(unit 1)
 				)
@@
 		(dnp no)
 		(fields_autoplaced yes)
-		(property "Reference" "#PWR053"
+		(property "Reference" "#PWR057"
 			(at 129.54 78.74 0)
 			(effects
@@
 			(project "Main PCB"
 				(path "/2fa7e914-8c49-49b7-a5a9-3cb78b2e953f/61c7190e-5a84-4d72-bf05-2bf9053a9edb"
-					(reference "#PWR053")
+					(reference "#PWR057")
 					(unit 1)
 				)
@@
 		(on_board yes)
 		(dnp no)
-		(property "Reference" "R26"
+		(property "Reference" "R41"
 			(at 160.02 66.04 0)
 			(effects
@@
 			(project "Main PCB"
 				(path "/2fa7e914-8c49-49b7-a5a9-3cb78b2e953f/61c7190e-5a84-4d72-bf05-2bf9053a9edb"
-					(reference "R26")
+					(reference "R41")
 					(unit 1)
 				)
@@
 		(on_board yes)
 		(dnp no)
-		(property "Reference" "R24"
+		(property "Reference" "R39"
 			(at 160.02 48.26 0)
 			(effects
@@
 			(project "Main PCB"
 				(path "/2fa7e914-8c49-49b7-a5a9-3cb78b2e953f/61c7190e-5a84-4d72-bf05-2bf9053a9edb"
-					(reference "R24")
+					(reference "R39")
 					(unit 1)
 				)
@@
 		(on_board yes)
 		(dnp no)
-		(property "Reference" "R22"
+		(property "Reference" "R37"
 			(at 160.02 30.48 0)
 			(effects
@@
 			(project "Main PCB"
 				(path "/2fa7e914-8c49-49b7-a5a9-3cb78b2e953f/61c7190e-5a84-4d72-bf05-2bf9053a9edb"
-					(reference "R22")
+					(reference "R37")
 					(unit 1)
 				)
@@
 		(on_board yes)
 		(dnp no)
-		(property "Reference" "R29"
+		(property "Reference" "R44"
 			(at 160.02 92.71 0)
 			(effects
@@
 			(project "Main PCB"
 				(path "/2fa7e914-8c49-49b7-a5a9-3cb78b2e953f/61c7190e-5a84-4d72-bf05-2bf9053a9edb"
-					(reference "R29")
+					(reference "R44")
 					(unit 1)
 				)
@@
 		(on_board yes)
 		(dnp no)
-		(property "Reference" "R20"
+		(property "Reference" "R35"
 			(at 107.188 84.328 90)
 			(effects
@@
 			(project "Main PCB"
 				(path "/2fa7e914-8c49-49b7-a5a9-3cb78b2e953f/61c7190e-5a84-4d72-bf05-2bf9053a9edb"
-					(reference "R20")
+					(reference "R35")
 					(unit 1)
 				)
@@
 		(on_board yes)
 		(dnp no)
-		(property "Reference" "R27"
+		(property "Reference" "R42"
 			(at 160.02 74.93 0)
 			(effects
@@
 			(project "Main PCB"
 				(path "/2fa7e914-8c49-49b7-a5a9-3cb78b2e953f/61c7190e-5a84-4d72-bf05-2bf9053a9edb"
-					(reference "R27")
+					(reference "R42")
 					(unit 1)
 				)
@@
 		(on_board yes)
 		(dnp no)
-		(property "Reference" "R19"
+		(property "Reference" "R34"
 			(at 107.188 76.708 90)
 			(effects
@@
 			(project "Main PCB"
 				(path "/2fa7e914-8c49-49b7-a5a9-3cb78b2e953f/61c7190e-5a84-4d72-bf05-2bf9053a9edb"
-					(reference "R19")
+					(reference "R34")
 					(unit 1)
 				)
@@
 		(on_board yes)
 		(dnp no)
-		(property "Reference" "R28"
+		(property "Reference" "R43"
 			(at 160.02 83.82 0)
 			(effects
@@
 			(project "Main PCB"
 				(path "/2fa7e914-8c49-49b7-a5a9-3cb78b2e953f/61c7190e-5a84-4d72-bf05-2bf9053a9edb"
-					(reference "R28")
+					(reference "R43")
 					(unit 1)
 				)
@@
 		(dnp no)
 		(fields_autoplaced yes)
-		(property "Reference" "#PWR054"
+		(property "Reference" "#PWR058"
 			(at 129.54 86.36 0)
 			(effects
@@
 			(project "Main PCB"
 				(path "/2fa7e914-8c49-49b7-a5a9-3cb78b2e953f/61c7190e-5a84-4d72-bf05-2bf9053a9edb"
-					(reference "#PWR054")
+					(reference "#PWR058")
 					(unit 1)
 				)
@@
 		(dnp no)
 		(fields_autoplaced yes)
-		(property "Reference" "#PWR050"
+		(property "Reference" "#PWR054"
 			(at 107.95 60.96 0)
 			(effects
@@
 			(project "Main PCB"
 				(path "/2fa7e914-8c49-49b7-a5a9-3cb78b2e953f/61c7190e-5a84-4d72-bf05-2bf9053a9edb"
-					(reference "#PWR050")
+					(reference "#PWR054")
 					(unit 1)
 				)
@@
 		(dnp no)
 		(fields_autoplaced yes)
-		(property "Reference" "#PWR056"
+		(property "Reference" "#PWR060"
 			(at 184.15 63.5 0)
 			(effects
@@
 			(project "Main PCB"
 				(path "/2fa7e914-8c49-49b7-a5a9-3cb78b2e953f/61c7190e-5a84-4d72-bf05-2bf9053a9edb"
-					(reference "#PWR056")
+					(reference "#PWR060")
 					(unit 1)
 				)
@@
 		(dnp no)
 		(fields_autoplaced yes)
-		(property "Reference" "#PWR049"
+		(property "Reference" "#PWR053"
 			(at 107.95 45.72 0)
 			(effects
@@
 			(project "Main PCB"
 				(path "/2fa7e914-8c49-49b7-a5a9-3cb78b2e953f/61c7190e-5a84-4d72-bf05-2bf9053a9edb"
-					(reference "#PWR049")
+					(reference "#PWR053")
 					(unit 1)
 				)
@@
 		(dnp no)
 		(fields_autoplaced yes)
-		(property "Reference" "#PWR048"
+		(property "Reference" "#PWR052"
 			(at 107.95 38.1 0)
 			(effects
@@
 			(project "Main PCB"
 				(path "/2fa7e914-8c49-49b7-a5a9-3cb78b2e953f/61c7190e-5a84-4d72-bf05-2bf9053a9edb"
-					(reference "#PWR048")
+					(reference "#PWR052")
 					(unit 1)
 				)
@@
 		(on_board yes)
 		(dnp no)
-		(property "Reference" "R18"
+		(property "Reference" "R33"
 			(at 107.95 59.69 0)
 			(effects
@@
 			(project "Main PCB"
 				(path "/2fa7e914-8c49-49b7-a5a9-3cb78b2e953f/61c7190e-5a84-4d72-bf05-2bf9053a9edb"
-					(reference "R18")
+					(reference "R33")
 					(unit 1)
 				)
@@
 		(on_board yes)
 		(dnp no)
-		(property "Reference" "R25"
+		(property "Reference" "R40"
 			(at 160.02 57.15 0)
 			(effects
@@
 			(project "Main PCB"
 				(path "/2fa7e914-8c49-49b7-a5a9-3cb78b2e953f/61c7190e-5a84-4d72-bf05-2bf9053a9edb"
-					(reference "R25")
+					(reference "R40")
 					(unit 1)
 				)
@@
 		(dnp no)
 		(fields_autoplaced yes)
-		(property "Reference" "#PWR055"
+		(property "Reference" "#PWR059"
 			(at 129.54 93.98 0)
 			(effects
@@
 			(project "Main PCB"
 				(path "/2fa7e914-8c49-49b7-a5a9-3cb78b2e953f/61c7190e-5a84-4d72-bf05-2bf9053a9edb"
-					(reference "#PWR055")
+					(reference "#PWR059")
 					(unit 1)
 				)
@@
 		(on_board yes)
 		(dnp no)
-		(property "Reference" "R23"
+		(property "Reference" "R38"
 			(at 160.02 39.37 0)
 			(effects
@@
 			(project "Main PCB"
 				(path "/2fa7e914-8c49-49b7-a5a9-3cb78b2e953f/61c7190e-5a84-4d72-bf05-2bf9053a9edb"
-					(reference "R23")
+					(reference "R38")
 					(unit 1)
 				)
@@
 		(dnp no)
 		(fields_autoplaced yes)
-		(property "Reference" "#PWR051"
+		(property "Reference" "#PWR055"
 			(at 129.54 53.34 0)
 			(effects
@@
 			(project "Main PCB"
 				(path "/2fa7e914-8c49-49b7-a5a9-3cb78b2e953f/61c7190e-5a84-4d72-bf05-2bf9053a9edb"
-					(reference "#PWR051")
+					(reference "#PWR055")
 					(unit 1)
 				)
@@
 		(on_board yes)
 		(dnp no)
-		(property "Reference" "R17"
+		(property "Reference" "R32"
 			(at 107.95 52.07 0)
 			(effects
@@
 			(project "Main PCB"
 				(path "/2fa7e914-8c49-49b7-a5a9-3cb78b2e953f/61c7190e-5a84-4d72-bf05-2bf9053a9edb"
-					(reference "R17")
-					(unit 1)
-				)
+					(reference "R32")
+					(unit 1)
+				)
